File: SnarkBarker.kicad_pcb (KiCad board)
At the start: 2 copper layers, 231.1 x 106.7 mm, 199 parts, among them J1 Bus_ISA_8bit, J2 Bracket Mount, P1 Joystick/MIDI, P2 L7809, T1 2N3904, T2 2N3904, U1 NE558, U10 YM3014B, U11 NJM3403A, U12 MC1408_DIP, U13 805X, U14 SAA1099, U15 SAA1099, U16 74LS08, U17 74LS139, U18 74LS374, U19 74LS374, U2 74LS245, U20 74LS74, U21 74LS125, U22 74LS74, U23 74LS74, U24 74LS32, U25 74LS08, U26 74LS74, U27 74LS32, U28 74LS08, U29 74LS14, U3 74LS244, U30 74LS32, U4 TEA2025B, U5 LM324, U6 LM393, U7 74LS138, U8 74LS138, U9 YM3812

Commit message: Add files via upload
Parts:
- removed the G*** at (106.5, 30.3)
- added G***: LOGO, SoundBlaster:Shark_Barber_Back, F.Cu at (107.6, 30.6)
- added REF**: Shark_Barber_Graphic, SoundBlaster:Shark_Barber_Graphic, F.Cu at (109.0, 53.7)
Other:
- board text added: ""Why do you have all these old computer parts?""
- board text added: "2021 Derivative Labs"
- board text added: "CC-BY-SA"
- board text added: "CREDITS:"
- board text added: "Lord_Nightmare, balrog, kevtris: lots of info Foone: testing (hi gewt)"
- board text added: "MADE IN HUNGER"
- board text added: "Special thanks: ##yamahasynths SHOUTS TO cr1901, CommodoreZ, glitch, Trixter"
- board text added: "TubeTimeUS: PCB reversing,"
- board text added: "forwarding, firmware analysis"
- board text removed: "CC BY-SA (Attribution-ShareAlike)"
- board text removed: "CREDITS"
- board text removed: "Foone: testing"
- board text removed: "Lord_Nightmare, balrog, kevtris: lots of info"
- board text removed: "MADE IN ANGER"
- board text removed: "SHOUTS TO cr1901, CommodoreZ, glitch, and Trixter"
- board text removed: "Special thanks to ##yamahasynths"
- board text removed: "TubeTimeUS: PCB reversing and forwarding,"
- board text removed: "also firmware analysis"
